Commit message: Sim working v1.02

File: urdf/apriltag_marker.urdf.xacro (robot description, xacro)
@@ -1,5 +1,4 @@
 <?xml version="1.0" ?>
-<robot xmlns:xacro="http://www.ros.org/wiki/xacro"
-       name="apriltag_marker">
+<robot name="apriltag_marker" xmlns:xacro="http://www.ros.org/wiki/xacro">
   <!-- ROS xacro/urdf model of one apriltag marker with given
        tag-family, ID, and size of the mesh. Optionally, apriltag_size can be
@@ -40,5 +39,5 @@
        </xacro:apriltag_marker>
    -->
-  <xacro:macro name="apriltag_marker" params="namespace name parent family ID size:=0 apriltag_size:=0 *origin" >
+  <xacro:macro name="apriltag_marker" params="namespace name ID size:=0 apriltag_size:=0 *origin" >
     <!-- Check in which way the size was specified -->
     <xacro:if value="${apriltag_size == 0}">
@@ -46,12 +45,7 @@
     </xacro:if>
     <xacro:if value="${apriltag_size != 0}">
-      <xacro:if value="${family == '36h11'}">
-        <xacro:property name="mesh_size" value="${apriltag_size/8*10}" />
-      </xacro:if>
-      <xacro:if value="${family == '16h5'}">
-        <xacro:property name="mesh_size" value="${apriltag_size/6*8}" />
-      </xacro:if>
+      <xacro:property name="mesh_size" value="${apriltag_size/8*10}" />
     </xacro:if>
-    <link name="${namespace}${name}">
+    <link name="${namespace}/${name}">
       <inertial>
         <mass value="0.001" />
@@ -69,10 +63,10 @@
         <geometry>
           <!-- use Python str to convert family name and to generate leading zeros -->
-          <mesh filename="$(find CRoCS)/meshes/tag${str(family).replace( 'h', '_' )}_${str(ID).zfill(5)}.dae" scale="${10*mesh_size} ${10*mesh_size} 1"/>
+          <mesh filename="file:///$(find CRoCS)/meshes/tag36_11_${str(ID).zfill(5)}.dae" scale="${10*mesh_size} ${10*mesh_size} 1"/>
         </geometry>
       </visual>
     </link>
     <!-- we use Gazebo material to put the texture onto the marker. Note mu1=mu2=0 for no friction. -->
-    <gazebo reference="${namespace}${name}">
+    <gazebo reference="${namespace}/${name}">
       <!-- <material>Gazebo/Red</material> -->
       <turnGravityOff>false</turnGravityOff>
@@ -83,8 +77,8 @@
       <kd>1.0</kd>
     </gazebo>
-    <joint name="${namespace}${name}_joint" type="fixed">
+    <joint name="${namespace}/${name}_joint" type="fixed">
       <xacro:insert_block name="origin" />
-      <parent link="${namespace}${parent}" />
-      <child link="${namespace}${name}" />
+      <parent link="${namespace}" />
+      <child link="${namespace}/${name}" />
     </joint>
   </xacro:macro>

File: urdf/cube.urdf.xacro (robot description, xacro)
@@ -1,55 +1,28 @@
 <?xml version="1.0"?>
 <robot name="cube" xmlns:xacro="http://www.ros.org/wiki/xacro">
-  <xacro:property name="caster_radius" value="0.006"/>
-  <xacro:property name="caster_mass" value="0.1"/>
-  <xacro:property name="caster_offset_back" value="-0.0508"/>
   <xacro:include filename="$(find CRoCS)/urdf/cube_macro.xacro"/>
-  <xacro:include filename="$(find CRoCS)/urdf/camera.xacro"/>
+  <!-- <xacro:include filename="$(find CRoCS)/urdf/camera.xacro"/> -->
   <xacro:include filename="$(find CRoCS)/urdf/apriltag_marker.urdf.xacro" />
+  <xacro:arg name="robot_name" default="cube1"/>
   <!-- Add cube -->
-  <xacro:cube/>
+  <xacro:cube name="$(arg robot_name)"/>
   <!-- Add April Tags -->
-  <!-- left -->
-  <xacro:apriltag_marker namespace="" name="$cube_tag_01" parent="cube"
-           family="36h11" ID="01" size="0.15243">
-           <origin xyz="0 ${0.15243/2 + 0.001} ${0.15243/2 + 0.004}" rpy="1.571 0 0" />
+  <xacro:apriltag_marker namespace="$(arg robot_name)" name="left_tag_01" ID="01" size="0.15243">
+    <origin xyz="0 ${0.15243/2 + 0.001} ${0.15243/2 + 0.004}" rpy="${pi/2} 0 0" />
   </xacro:apriltag_marker>
-  <!-- right -->
-  <xacro:apriltag_marker namespace="" name="$cube_tag_02" parent="cube"
-           family="36h11" ID="02" size="0.15243">
-           <origin xyz="0 ${-(0.15243/2 + 0.001)} ${0.15243/2 + 0.004}" rpy="-1.571 0 0" />
+  <xacro:apriltag_marker namespace="$(arg robot_name)" name="right_tag_02" ID="02" size="0.15243">
+    <origin xyz="0 ${-(0.15243/2 + 0.001)} ${0.15243/2 + 0.004}" rpy="${-pi/2} 0 0" />
   </xacro:apriltag_marker>
   <!-- Add wheels -->
-  <xacro:wheel direction="left"/>
-  <xacro:wheel direction="right"/>
-  <link name="caster">
-    <visual>
-      <geometry>
-        <sphere radius="${caster_radius}"/>
-      </geometry>
-    </visual>
-    <collision>
-      <geometry>
-        <sphere radius="${caster_radius}"/>
-      </geometry>
-    </collision>
-    <xacro:caster_intertial mass="${caster_mass}" radius="${caster_radius}"/>
-  </link>
-  <joint name="base_to_caster" type="fixed">
-    <parent link="cube"/>
-    <child link="caster"/>
-    <origin xyz="${caster_offset_back} 0 0"/>
-  </joint>
-  <gazebo reference="caster">
-    <mu1 value="0.0"/>
-    <mu2 value="0.0"/>
-    <kp value="10000000.0" />
-    <kd value="1.0" />
-    <material>Gazebo/Grey</material>
-  </gazebo>
+  <xacro:wheel  direction="left" name="$(arg robot_name)"/>
+  <xacro:wheel  direction="right" name="$(arg robot_name)"/>
+  <!-- Add caster -->
+  <xacro:caster name="$(arg robot_name)"/>
+  <!-- Add camera-->
+  <xacro:cam name="$(arg robot_name)"/>
   <!-- Gazebo plugin for ROS Control -->
   <gazebo>
     <plugin name="gazebo_ros_control" filename="libgazebo_ros_control.so">
-      <robotNamespace>/</robotNamespace>
+      <robotNamespace></robotNamespace>
     </plugin>
   </gazebo>

File: urdf/cube_macro.xacro (robot description, xacro)
@@ -1,4 +1,4 @@
 <?xml version="1.0"?>
-<robot name="cube" xmlns:xacro="http://www.ros.org/wiki/xacro">
+<robot xmlns:xacro="http://www.ros.org/wiki/xacro">
   <!-- Set constants -->
   <!-- Mass in kg, distance in meter -->
@@ -11,4 +11,7 @@
   <xacro:property name="wheel_offset_forward" value="0.033966"/>
   <xacro:property name="wheel_offset_side" value="0.05041"/>
+  <xacro:property name="caster_radius" value="0.006"/>
+  <xacro:property name="caster_mass" value="0.1"/>
+  <xacro:property name="caster_offset_back" value="-0.0508"/>
   <!-- Intertial for cube -->
   <xacro:macro name="cube_inertial">
@@ -26,17 +29,17 @@
   </xacro:macro>
   <!-- Intertial for sphere -->
-  <xacro:macro name="caster_intertial" params="mass radius">
+  <xacro:macro name="caster_intertial">
     <inertial>
-      <mass value="${mass}"/>
-      <inertia ixx="${2 * mass / 5 * radius*radius}" iyy="${2 * mass / 5 * radius*radius}" izz="${2 * mass / 5 * radius*radius}" ixy="0.0" ixz="0.0" iyz="0.0"/>
+      <mass value="${caster_mass}"/>
+      <inertia ixx="${2 * caster_mass / 5 * caster_radius*caster_radius}" iyy="${2 * caster_mass / 5 * caster_radius*caster_radius}" izz="${2 * caster_mass / 5 * caster_radius*caster_radius}" ixy="0.0" ixz="0.0" iyz="0.0"/>
     </inertial>
   </xacro:macro>
   <!-- Create cube -->
-  <xacro:macro name="cube">
+  <xacro:macro name="cube" params="name">
     <!-- Dummy to attach cube to and get rid of warning and stuffs -->
-    <link name="dummy">
+    <link name="${name}_dummy">
     </link>
     <!-- Build cube shape -->
-    <link name="cube">
+    <link name="${name}">
       <visual>
         <geometry>
@@ -54,13 +57,14 @@
       <xacro:cube_inertial/>
     </link>
-    <joint name="dummy_joint" type="fixed">
-      <parent link="dummy"/>
-      <child link="cube"/>
+    <joint name="${name}_dummy_joint" type="fixed">
+      <parent link="${name}_dummy"/>
+      <child link="${name}"/>
+      <origin xyz="0 0 0"/>
     </joint>
   </xacro:macro>
   <!-- Create wheel -->
-  <xacro:macro name="wheel" params="direction">
+  <xacro:macro name="wheel" params="direction name">
     <!-- Build the shape -->
-    <link name="${direction}_wheel">
+    <link name="${name}_${direction}_wheel">
       <visual>
         <geometry>
@@ -78,5 +82,5 @@
     </link>
     <!-- Add gazebo physics -->
-    <gazebo reference="${direction}_wheel">
+    <gazebo reference="${name}_${direction}_wheel">
       <mu1 value="200.0"/>
       <mu2 value="100.0"/>
@@ -86,7 +90,7 @@
     </gazebo>
     <!-- Attach to cube accordingly based on left/right wheel -->
-    <joint name="${direction}_wheel_joint" type="continuous">
-      <parent link="cube"/>
-      <child link="${direction}_wheel"/>
+    <joint name="${name}_${direction}_wheel_joint" type="continuous">
+      <parent link="${name}"/>
+      <child link="${name}_${direction}_wheel"/>
       <xacro:if value="${direction=='left'}">
         <origin xyz="${wheel_offset_forward} ${wheel_offset_side} ${wheel_offset_up}"/>
@@ -98,13 +102,90 @@
     </joint>
     <!-- For control -->
-    <transmission name="${direction}_wheel_trans">
+    <transmission name="${name}_${direction}_wheel_trans">
       <type>transmission_interface/SimpleTransmission</type>
-      <actuator name="${direction}_wheel_motor">
+      <actuator name="${name}_${direction}_wheel_motor">
         <mechanicalReduction>1</mechanicalReduction>
       </actuator>
-      <joint name="${direction}_wheel_joint">
+      <joint name="${name}_${direction}_wheel_joint">
         <hardwareInterface>hardware_interface/VelocityJointInterface</hardwareInterface>
       </joint>
     </transmission>
   </xacro:macro>
+  <!-- Create caster -->
+  <xacro:macro name="caster" params="name">
+    <link name="${name}_caster">
+      <visual>
+        <geometry>
+          <sphere radius="${caster_radius}"/>
+        </geometry>
+      </visual>
+      <collision>
+        <geometry>
+          <sphere radius="${caster_radius}"/>
+        </geometry>
+      </collision>
+      <xacro:caster_intertial/>
+    </link>
+    <joint name="${name}_to_caster" type="fixed">
+      <parent link="${name}"/>
+      <child link="${name}_caster"/>
+      <origin xyz="${caster_offset_back} 0 0"/>
+    </joint>
+    <gazebo reference="${name}_caster">
+      <mu1 value="0.0"/>
+      <mu2 value="0.0"/>
+      <kp value="10000000.0" />
+      <kd value="1.0" />
+      <material>Gazebo/Grey</material>
+    </gazebo>
+  </xacro:macro>
+  <!-- Create camera -->
+  <xacro:macro name="cam" params="name">
+      <link name="${name}_camera_link">
+          <visual>
+              <geometry>
+                  <box size="0.010 0.03 0.03"/>
+              </geometry>
+          </visual>
+      </link>
+      <joint name="${name}_camera_joint" type="fixed">
+          <parent link="${name}"/>
+          <child link="${name}_camera_link"/>
+          <origin xyz="0.0762 0 0.0762" rpy="0 0 0"/>
+      </joint>
+      <link name="${name}_camera_link_optical"></link>
+      <joint name="${name}_camera_optical_joint" type="fixed">
+          <parent link="${name}_camera_link"/>
+          <child link="${name}_camera_link_optical"/>
+          <origin xyz="0 0 0" rpy="${-pi/2} 0 ${-pi/2}"/>
+      </joint>
+      <gazebo reference="${name}_camera_link">
+          <material>Gazebo/Red</material>
+          <sensor name="${name}_cam" type="camera">
+              <pose> 0 0 0 0 0 0 </pose>
+              <visualize>true</visualize>
+              <update_rate>10</update_rate>
+              <camera>
+                  <horizontal_fov>1.0821</horizontal_fov>
+                  <vertical_fov>0.820305</vertical_fov>
+                  <image>
+                      <format>R8G8B8</format>
+                      <width>640</width>
+                      <height>480</height>
+                  </image>
+                  <clip>
+                      <near>0.05</near>
+                      <far>8.0</far>
+                  </clip>
+              </camera>
+              <plugin name="${name}_camera_controller" filename="libgazebo_ros_camera.so">
+                  <cameraName>${name}/camera</cameraName>
+                  <imageTopicName>image_raw</imageTopicName>
+                  <cameraInfoTopicName>camera_info</cameraInfoTopicName>
+                  <frameName>${name}_camera_link</frameName>
+                  <!-- <frame_name>camera_link_optical</frame_name> -->
+              </plugin>
+          </sensor>
+      </gazebo>
+  </xacro:macro>
 </robot>

Commit message: Test kalman, simulate true and kalman path in rviz

File: urdf/apriltag_marker.urdf.xacro (robot description, xacro)
@@ -63,5 +63,5 @@
         <geometry>
           <!-- use Python str to convert family name and to generate leading zeros -->
-          <mesh filename="file:///$(find CRoCS)/meshes/tag36_11_${str(ID).zfill(5)}.dae" scale="${10*mesh_size} ${10*mesh_size} 1"/>
+          <mesh filename="file:///$(find CRoCS)/models/tag36_11_${str(ID).zfill(5)}.dae" scale="${10*mesh_size} ${10*mesh_size} 1"/>
         </geometry>
       </visual>

File: urdf/cube.urdf.xacro (robot description, xacro)
@@ -17,25 +17,4 @@
     <origin xyz="0 ${-(0.15243/2 + 0.001)} ${0.15243/2 + 0.004}" rpy="${-pi/2} ${pi}  ${pi} " />
   </xacro:apriltag_marker>
-  <!-- <model name='Apriltag36_11_00000'>
-    <link name='main'>
-      <pose>0 0 0 0 -0 0</pose>
-      <visual name='main_Visual'>
-        <geometry>
-          <box>
-            <size>1 1 0.01</size>
-          </box>
-        </geometry>
-        <material>
-          <script>
-            <uri>model://Apriltag36_11_00000/materials/scripts</uri>
-            <uri>model://Apriltag36_11_00000/materials/textures</uri>
-            <name>Apriltag36_11_00000</name>
-          </script>
-        </material>
-      </visual>
-    </link>
-    <static>1</static>
-    <pose>4.05194 0.010848 0 0 -0 0</pose>
-  </model> -->
   <!-- Add wheels -->
   <xacro:wheel  direction="left" name="$(arg robot_name)"/>
