Commit message: Multi cube sim working

File: urdf/cube.urdf.xacro (robot description, xacro)
@@ -5,4 +5,7 @@
   <xacro:include filename="$(find CRoCS)/urdf/apriltag_marker.urdf.xacro" />
   <xacro:arg name="robot_name" default="cube1"/>
+  <xacro:arg name="rotate" default="0.0"/>
+  <xacro:property name="temp" value="$(arg rotate)"/>
+  <xacro:property name="rotate" value="${temp * pi / 180}"/>
   <!-- Add cube -->
   <xacro:cube name="$(arg robot_name)"/>
@@ -24,5 +27,6 @@
   <gazebo>
     <plugin name="gazebo_ros_control" filename="libgazebo_ros_control.so">
-      <robotNamespace></robotNamespace>
+      <robotNamespace>/$(arg robot_name)</robotNamespace>
+      <robotParam>$(arg robot_name)/robot_description</robotParam>
     </plugin>
   </gazebo>

File: urdf/cube_macro.xacro (robot description, xacro)
@@ -47,5 +47,5 @@
         </geometry>
         <!-- Lift it up a bit to avoid clipping -->
-        <origin xyz="0 0 0.08"/>
+        <origin xyz="0 0 0.08" />
       </visual>
       <collision>
@@ -53,5 +53,5 @@
           <box size="${cube_length} ${cube_length} ${cube_length}"/>
         </geometry>
-        <origin xyz="0 0 0.08"/>
+        <origin xyz="0 0 0.08" />
       </collision>
       <xacro:cube_inertial/>
@@ -60,5 +60,6 @@
       <parent link="${name}_dummy"/>
       <child link="${name}"/>
-      <origin xyz="0 0 0"/>
+      <!-- Rotate the robot by (rotate) degrees, after converting it to radians -->
+      <origin xyz="0 0 0" rpy="0 0 ${rotate}"/>
     </joint>
   </xacro:macro>
@@ -94,8 +95,8 @@
       <child link="${name}_${direction}_wheel"/>
       <xacro:if value="${direction=='left'}">
-        <origin xyz="${wheel_offset_forward} ${wheel_offset_side} ${wheel_offset_up}"/>
+        <origin xyz="${wheel_offset_forward} ${wheel_offset_side} ${wheel_offset_up}" />
       </xacro:if>
       <xacro:if value="${direction=='right'}">
-        <origin xyz="${wheel_offset_forward} ${-wheel_offset_side} ${wheel_offset_up}"/>
+        <origin xyz="${wheel_offset_forward} ${-wheel_offset_side} ${wheel_offset_up}" />
       </xacro:if>
       <axis xyz="0 1 0"/>
@@ -130,5 +131,5 @@
       <parent link="${name}"/>
       <child link="${name}_caster"/>
-      <origin xyz="${caster_offset_back} 0 0"/>
+      <origin xyz="${caster_offset_back} 0 0" />
     </joint>
     <gazebo reference="${name}_caster">
@@ -152,5 +153,5 @@
           <parent link="${name}"/>
           <child link="${name}_camera_link"/>
-          <origin xyz="0.0762 0 0.0762" rpy="0 0 0"/>
+          <origin xyz="0.0762 0 0.0762" />
       </joint>
       <link name="${name}_camera_link_optical"></link>
@@ -180,5 +181,5 @@
               </camera>
               <plugin name="${name}_camera_controller" filename="libgazebo_ros_camera.so">
-                  <cameraName>${name}/camera</cameraName>
+                  <cameraName>camera</cameraName>
                   <imageTopicName>image_raw</imageTopicName>
                   <cameraInfoTopicName>camera_info</cameraInfoTopicName>

Commit message: Sim can spawn multiple cubes and detect april tags on each cube sides

File: urdf/cube.urdf.xacro (robot description, xacro)
@@ -11,10 +11,31 @@
   <xacro:cube name="$(arg robot_name)"/>
   <!-- Add April Tags -->
-  <xacro:apriltag_marker namespace="$(arg robot_name)" name="left_tag_01" ID="01" size="0.15243">
-    <origin xyz="0 ${0.15243/2 + 0.001} ${0.15243/2 + 0.004}" rpy="${pi/2} 0 0" />
+  <xacro:apriltag_marker namespace="$(arg robot_name)" name="left_tag_05" ID="05" size="0.15243">
+    <origin xyz="0 ${0.15243/2 + 0.001} ${0.15243/2 + 0.004}" rpy="${pi/2} 0 ${pi} " />
   </xacro:apriltag_marker>
-  <xacro:apriltag_marker namespace="$(arg robot_name)" name="right_tag_02" ID="02" size="0.15243">
-    <origin xyz="0 ${-(0.15243/2 + 0.001)} ${0.15243/2 + 0.004}" rpy="${-pi/2} 0 0" />
+  <xacro:apriltag_marker namespace="$(arg robot_name)" name="right_tag_05" ID="05" size="0.15243">
+    <origin xyz="0 ${-(0.15243/2 + 0.001)} ${0.15243/2 + 0.004}" rpy="${-pi/2} ${pi}  ${pi} " />
   </xacro:apriltag_marker>
+  <!-- <model name='Apriltag36_11_00000'>
+    <link name='main'>
+      <pose>0 0 0 0 -0 0</pose>
+      <visual name='main_Visual'>
+        <geometry>
+          <box>
+            <size>1 1 0.01</size>
+          </box>
+        </geometry>
+        <material>
+          <script>
+            <uri>model://Apriltag36_11_00000/materials/scripts</uri>
+            <uri>model://Apriltag36_11_00000/materials/textures</uri>
+            <name>Apriltag36_11_00000</name>
+          </script>
+        </material>
+      </visual>
+    </link>
+    <static>1</static>
+    <pose>4.05194 0.010848 0 0 -0 0</pose>
+  </model> -->
   <!-- Add wheels -->
   <xacro:wheel  direction="left" name="$(arg robot_name)"/>

Commit message: Sim sim sim

File: urdf/cube.urdf.xacro (robot description, xacro)
@@ -11,9 +11,12 @@
   <xacro:cube name="$(arg robot_name)"/>
   <!-- Add April Tags -->
-  <xacro:apriltag_marker namespace="$(arg robot_name)" name="left_tag_05" ID="05" size="0.15243">
+  <xacro:apriltag_marker namespace="$(arg robot_name)" name="left_tag_11" ID="11" size="0.15243">
     <origin xyz="0 ${0.15243/2 + 0.001} ${0.15243/2 + 0.004}" rpy="${pi/2} 0 ${pi} " />
   </xacro:apriltag_marker>
-  <xacro:apriltag_marker namespace="$(arg robot_name)" name="right_tag_05" ID="05" size="0.15243">
+  <xacro:apriltag_marker namespace="$(arg robot_name)" name="right_tag_11" ID="11" size="0.15243">
     <origin xyz="0 ${-(0.15243/2 + 0.001)} ${0.15243/2 + 0.004}" rpy="${-pi/2} ${pi}  ${pi} " />
+  </xacro:apriltag_marker>
+  <xacro:apriltag_marker namespace="$(arg robot_name)" name="front_tag_10" ID="10" size="0.0254">
+    <origin xyz="${-(0.15243/2 + 0.001)} 0 ${0.15243/2 + 0.004}" rpy="0 ${pi/2}  ${pi} " />
   </xacro:apriltag_marker>
   <!-- Add wheels -->

File: urdf/cube_macro.xacro (robot description, xacro)
@@ -9,5 +9,5 @@
   <xacro:property name="wheel_mass" value="0.1"/>
   <xacro:property name="wheel_offset_up" value="0.015243"/>
-  <xacro:property name="wheel_offset_forward" value="0.033966"/>
+  <xacro:property name="wheel_offset_forward" value="0.039624"/>
   <xacro:property name="wheel_offset_side" value="0.05041"/>
   <xacro:property name="caster_radius" value="0.006"/>

Commit message: CBS Path planning V0.8

File: urdf/cube.urdf.xacro (robot description, xacro)
@@ -6,4 +6,8 @@
   <xacro:arg name="robot_name" default="cube1"/>
   <xacro:arg name="rotate" default="0.0"/>
+  <xacro:arg name="side" default="00"/>
+  <xacro:arg name="back" default="01"/>
+  <xacro:arg name="frontleft" default="02"/>
+  <xacro:arg name="frontright" default="03"/>
   <xacro:property name="temp" value="$(arg rotate)"/>
   <xacro:property name="rotate" value="${temp * pi / 180}"/>
@@ -11,12 +15,18 @@
   <xacro:cube name="$(arg robot_name)"/>
   <!-- Add April Tags -->
-  <xacro:apriltag_marker namespace="$(arg robot_name)" name="left_tag_11" ID="11" size="0.15243">
+  <xacro:apriltag_marker namespace="$(arg robot_name)" name="left_tag_$(arg side)" ID="$(arg side)" size="0.15243">
     <origin xyz="0 ${0.15243/2 + 0.001} ${0.15243/2 + 0.004}" rpy="${pi/2} 0 ${pi} " />
   </xacro:apriltag_marker>
-  <xacro:apriltag_marker namespace="$(arg robot_name)" name="right_tag_11" ID="11" size="0.15243">
+  <xacro:apriltag_marker namespace="$(arg robot_name)" name="right_tag_$(arg side)" ID="$(arg side)" size="0.15243">
     <origin xyz="0 ${-(0.15243/2 + 0.001)} ${0.15243/2 + 0.004}" rpy="${-pi/2} ${pi}  ${pi} " />
   </xacro:apriltag_marker>
-  <xacro:apriltag_marker namespace="$(arg robot_name)" name="front_tag_10" ID="10" size="0.0254">
-    <origin xyz="${-(0.15243/2 + 0.001)} 0 ${0.15243/2 + 0.004}" rpy="0 ${pi/2}  ${pi} " />
+  <xacro:apriltag_marker namespace="$(arg robot_name)" name="back_tag_$(arg back)" ID="$(arg back)" size="0.0254">
+    <origin xyz="${-(0.15243/2 + 0.001)} 0 ${0.15243/2 + 0.004}" rpy="${pi/2} 0 ${-pi/2}" />
+  </xacro:apriltag_marker>
+  <xacro:apriltag_marker namespace="$(arg robot_name)" name="front_left_tag_$(arg frontleft)" ID="$(arg frontleft)" size="0.0254">
+    <origin xyz="${(0.15243/2 + 0.001)} ${0.15243/3} ${0.15243/2 + 0.004}" rpy="${pi/2} 0 ${pi/2}" />
+  </xacro:apriltag_marker>
+  <xacro:apriltag_marker namespace="$(arg robot_name)" name="front_right_tag_$(arg frontright)" ID="$(arg frontright)" size="0.0254">
+    <origin xyz="${(0.15243/2 + 0.001)} ${-0.15243/3}  ${0.15243/2 + 0.004}" rpy="${pi/2} 0 ${pi/2}" />
   </xacro:apriltag_marker>
   <!-- Add wheels -->

Commit message: Final demo sim

File: urdf/cube.urdf.xacro (robot description, xacro)
@@ -25,8 +25,8 @@
   </xacro:apriltag_marker>
   <xacro:apriltag_marker namespace="$(arg robot_name)" name="front_left_tag_$(arg frontleft)" ID="$(arg frontleft)" size="0.0254">
-    <origin xyz="${(0.15243/2 + 0.001)} ${0.15243/3} ${0.15243/2 + 0.004}" rpy="${pi/2} 0 ${pi/2}" />
+    <origin xyz="${(0.15243/2 + 0.001)} ${0.0346} ${0.15243/2 + 0.004}" rpy="${pi/2} 0 ${pi/2}" />
   </xacro:apriltag_marker>
   <xacro:apriltag_marker namespace="$(arg robot_name)" name="front_right_tag_$(arg frontright)" ID="$(arg frontright)" size="0.0254">
-    <origin xyz="${(0.15243/2 + 0.001)} ${-0.15243/3}  ${0.15243/2 + 0.004}" rpy="${pi/2} 0 ${pi/2}" />
+    <origin xyz="${(0.15243/2 + 0.001)} ${-0.0346}  ${0.15243/2 + 0.004}" rpy="${pi/2} 0 ${pi/2}" />
   </xacro:apriltag_marker>
   <!-- Add wheels -->
